Commit message: modified model to accomodate camera angle and changes to physical robot

File: urdf/robot.urdf (robot description, URDF)
Before this commit: robot robot, 6 links, 5 joints
Links:
- link front_left_wheel: geometry collision cylinder length=0.02 radius=0.05; visual cylinder length=0.01 radius=0.075
- link front_right_wheel: geometry collision cylinder length=0.02 radius=0.05; visual cylinder length=0.01 radius=0.075
Joints:
- joint front_base_to_left_wheel: origin xyz=0 -0.06 0 rpy=0 0 -1.57 -> xyz=0 -0.06 -0.025 rpy=0 0 -1.57
- joint front_base_to_right_wheel: origin xyz=0 0.06 0 rpy=0 0 1.57 -> xyz=0 0.06 -0.025 rpy=0 0 1.57
- joint robot_to_base: origin xyz=0.00 0 0.025 rpy=0 0 0 -> xyz=0.00 0 0.05 rpy=0 0 0
- joint top_to_usb_cam: origin xyz=0.06 0 0.03 rpy=-1.57 0 -1.57 -> xyz=0.06 0 0.03 rpy=-1.59 0 -1.57

Commit message: change the model wheels

File: urdf/robot.urdf (robot description, URDF)
Before this commit: robot robot, 6 links, 5 joints
Links:
- link front_left_wheel: geometry collision cylinder length=0.02 radius=0.05; visual cylinder length=0.01 radius=0.0375
- link front_right_wheel: geometry collision cylinder length=0.02 radius=0.05; visual cylinder length=0.01 radius=0.0375

Commit message: all links fixed

File: urdf/robot.urdf (robot description, URDF)
Before this commit: robot robot, 6 links, 5 joints
Joints:
- joint front_base_to_left_wheel: type continuous -> fixed
- joint front_base_to_right_wheel: type continuous -> fixed

Commit message: added caster to robot

File: urdf/robot.urdf (robot description, URDF)
Before this commit: robot robot, 6 links, 5 joints
Links:
- added link caster, mass 10; collision sphere radius=0.02; visual sphere radius=0.02
- link front_left_wheel: geometry collision cylinder length=0.02 radius=0.0375; visual cylinder length=0.01 radius=0.0375
- link front_right_wheel: geometry collision cylinder length=0.02 radius=0.0375; visual cylinder length=0.01 radius=0.0375
- link usb_cam: mass 10 -> 0
Joints:
- added joint base_to_caster: type fixed, parent base, child caster, origin xyz=-.06 0. -0.0375 rpy=0 0 0 , limit effort=100 velocity=100

Commit message: able to spawn model and control it with diff control. Motion is not perfect

File: urdf/robot.urdf (robot description, URDF)
Before this commit: robot robot, 7 links, 6 joints
Links:
- link base: mass 10 -> 1
- link caster: mass 10 -> 3
- link front_left_wheel: mass 0.05 -> 1.5
- link front_right_wheel: mass 0.05 -> 1.5
- link top: mass 10 -> 1
- link usb_cam: mass 0 -> 0.1
Joints:
- joint front_base_to_left_wheel: origin xyz=0 -0.06 -0.025 rpy=0 0 -1.57 -> xyz=0 -0.08 -0.02 rpy=0 0 1.57; type fixed -> continuous
- joint front_base_to_right_wheel: origin xyz=0 0.06 -0.025 rpy=0 0 1.57 -> xyz=0 0.08 -0.02 rpy=0 0 1.57; type fixed -> continuous
- joint top_to_usb_cam: origin xyz=0.06 0 0.03 rpy=-1.59 0 -1.57 -> xyz=0.06 0 0.05 rpy=0 0 0
